File: 8to4Stepper.kicad_pcb (KiCad board)
At the start: 2 copper layers, 50 x 21 mm, 6 parts, among them J1 Out, J2 In

Commit message: Add gerber files.
Parts:
- moved JP4 11.3 mm to (200.0, 117.8)
- moved JP2 11.1 mm to (196.2, 112.8)
- moved J1 10.8 mm to (204.8, 124.5)
- moved JP3 5.15 mm to (200.0, 126.5)
- moved JP1 5.07 mm to (196.2, 121.5)
Routing:
- net /YEL: track 34.5 -> 15.8 mm, vias 1 -> 0
- net /BLK: track 34.3 -> 20.6 mm
- net /ORG: track 48.1 -> 35.6 mm, vias 1 -> 0
- net /PUR: track 19.9 -> 8.27 mm
- net /RED: track 28.9 -> 19.4 mm
- net /BLU: track 22.1 -> 19.1 mm
- net /BRN: track 18.5 -> 16.1 mm
- net /WHT: track 13.0 -> 10.7 mm
Other:
- board size 50 x 21 mm -> 32.2 x 18.5 mm
- board text added: "P"
- board text added: "S"
- board text removed: "Parallel"
- board text removed: "Serial"
