File: OpenDog_Teensy.kicad_pcb (KiCad board)
At the start: 2 copper layers, 61.6 x 96 mm, 62 parts, among them J1 NRF, J10 UART5, J11 UART6, J12 CAN1, J13 CAN2, J14 EXP, J15 Power, J2 TOF1, J3 TOF2, J4 IMU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

Commit message: Add more vias. Resolve DRC warnings.
Routing:
- net GND: vias 79 -> 106
Other:
- board text added: "(c) iQury.us Sep 2022"
- board text removed: "(c) iQury.us Aug 2022"

Commit message: OpenDog_Teensy - add buck converter socket. Move the battery monitor to the battery input instead of the 5V input in the old version.
Parts:
- added J16: VReg, Connector_PinSocket_2.54mm:PinSocket_1x04_P2.54mm_Vertical, F.Cu at (48.8, 129.4)
- moved C2 15.6 mm to (46.5, 131.1), turned to -90 degrees
Connections:
- C1 pad 1: /VIn -> /5V
- C2 pad 1: /VIn -> /5V
- C3 pad 1: /VIn -> /5V
- C4 pad 1: /VIn -> /5V
- C5 pad 1: /VIn -> /5V
- C6 pad 1: /VIn -> /5V
- J14 pad 2: /VIn -> /5V
- J15 pad 2: /VIn -> /Vbat
- R6 pad 1: /VIn -> /Vbat
- U1 pad 48: /VIn -> /5V
- U2 pad 3: /VIn -> /5V
- U3 pad 3: /VIn -> /5V
Routing:
- net /VIn: track 172.5 -> 0.00 mm, vias 1 -> 0
- net /5V: track 0.00 -> 166.2 mm, vias 0 -> 1
- net /Vbat: track 0.00 -> 33.4 mm
- net /3.3V: track 299.2 -> 300.0 mm, vias 2 -> 3
- net GND: vias 106 -> 107
Other:
- board text added: "6V-10V"
- board text added: "EN"
- board text added: "IN"
- board text added: "OpenDog V3 Teensy adapter V1c"
- board text added: "Out"
- board text added: "Power 6V-10V"
- board text removed: "5V"
- board text removed: "OpenDog V3 Teensy adapter V1b"
- board text removed: "Power 5V"

Commit message: OpenDog_Teensy - Update routing. Sent to fab.
Parts:
- R6: value 4.7k -> 82k
- R7: value 2.2k -> 22k
- moved C2 0.30 mm to (46.2, 131.1)
Routing:
- net GND: track 22.4 -> 27.9 mm, vias 107 -> 119
Other:
- board text added: "6V-15V"
- board text added: "Power 6V-15V"
- board text removed: "6V-10V"
- board text removed: "Power 6V-10V"
