File: OpenDog_Remote.kicad_sch (KiCad schematic)
At the start: 56 parts, among them J1 Conn_01x03_Pin, J10 Conn_01x03_Pin, J11 Conn_01x03_Pin, J12 Conn_01x02_Pin, J13 Conn_01x03_Pin, J14 Conn_01x03_Pin, J15 Conn_01x03_Pin, J16 Conn_01x03_Pin, J17 NRF, J18 Conn_02x08_Odd_Even, J2 Conn_01x03_Pin, J3 Conn_01x03_Pin, J4 Conn_01x03_Pin, J5 Conn_01x03_Pin, J6 Conn_01x03_Pin, J7 Conn_01x14, J8 Conn_01x03_Pin, J9 Conn_01x03_Pin, U1 Teensy4.1

Commit message: Separate screen and NRF/Touch SPI channels.
Connections:
- net B2: now also U1.2 (0_RX1_CRX2_CS1); no longer U1.18 (26_A12_MOSI1)
- net B2_LED: now also U1.24 (32_OUT1B); no longer U1.19 (27_A13_SCK1)
- net EX3: now also J18.7 (Pin_7); no longer J18.5 (Pin_5)
- net MISO: no longer J17.1 (Pin_1), J7.13 (Pin_13)
- net MOSI: no longer J17.4 (Pin_4), J7.12 (Pin_12)
- net SCK: no longer J17.3 (Pin_3), J7.10 (Pin_10)
- net EX1 renamed MOSI2
- net MOSI2: now also J17.4 (Pin_4), J7.12 (Pin_12), U1.18 (26_A12_MOSI1); no longer U1.2 (0_RX1_CRX2_CS1)
- net EX2 renamed MISO2
- net MISO2: now also J17.1 (Pin_1), J7.13 (Pin_13), U1.31 (39_MISO1_OUT1A); no longer U1.24 (32_OUT1B)
- removed net EX5: J18.7 (Pin_7), U1.31 (39_MISO1_OUT1A)
- new net SCK2: J17.3 (Pin_3), J18.5 (Pin_5), J7.10 (Pin_10), U1.19 (27_A13_SCK1)
Changed lines of the file:
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@@
     (stroke (width 0) (type default))
   )
-  (label "MISO" (at 26.035 116.205 0) (fields_autoplaced)
+  (label "MISO2" (at 26.035 116.205 0) (fields_autoplaced)
     (effects (font (size 1.27 1.27)) (justify left bottom))
   )
@@
     (effects (font (size 1.27 1.27)) (justify left bottom))
   )
-  (label "B2_LED" (at 73.025 88.265 0) (fields_autoplaced)
+  (label "B2_LED" (at 73.025 100.965 0) (fields_autoplaced)
     (effects (font (size 1.27 1.27)) (justify left bottom))
   )
@@
     (effects (font (size 1.27 1.27)) (justify left bottom))
   )
-  (label "EX3" (at 24.765 45.72 0) (fields_autoplaced)
+  (label "EX3" (at 24.765 48.26 0) (fields_autoplaced)
+    (effects (font (size 1.27 1.27)) (justify left bottom))
+  )
+  (label "MISO2" (at 140.97 85.725 0) (fields_autoplaced)
     (effects (font (size 1.27 1.27)) (justify left bottom))
   )
@@
     (effects (font (size 1.27 1.27)) (justify left bottom))
   )
-  (label "SCK" (at 184.15 139.065 0) (fields_autoplaced)
+  (label "SCK2" (at 184.15 139.065 0) (fields_autoplaced)
     (effects (font (size 1.27 1.27)) (justify left bottom))
   )
@@
     (effects (font (size 1.27 1.27)) (justify left bottom))
   )
-  (label "B2" (at 73.025 85.725 0) (fields_autoplaced)
+  (label "B2" (at 73.025 45.085 0) (fields_autoplaced)
     (effects (font (size 1.27 1.27)) (justify left bottom))
   )
@@
     (effects (font (size 1.27 1.27)) (justify left bottom))
   )
-  (label "EX1" (at 73.025 45.085 0) (fields_autoplaced)
-    (effects (font (size 1.27 1.27)) (justify left bottom))
-  )
   (label "Y2" (at 189.865 90.805 0) (fields_autoplaced)
     (effects (font (size 1.27 1.27)) (justify left bottom))
@@
     (effects (font (size 1.27 1.27)) (justify left bottom))
   )
-  (label "EX2" (at 46.99 43.18 0) (fields_autoplaced)
+  (label "MISO2" (at 45.085 43.18 0) (fields_autoplaced)
     (effects (font (size 1.27 1.27)) (justify left bottom))
   )
@@
     (effects (font (size 1.27 1.27)) (justify left bottom))
   )
-  (label "EX5" (at 142.875 85.725 0) (fields_autoplaced)
-    (effects (font (size 1.27 1.27)) (justify left bottom))
-  )
-  (label "EX2" (at 73.025 100.965 0) (fields_autoplaced)
-    (effects (font (size 1.27 1.27)) (justify left bottom))
-  )
   (label "~{TOUCH_CS}" (at 184.15 141.605 0) (fields_autoplaced)
     (effects (font (size 1.27 1.27)) (justify left bottom))
@@
     (effects (font (size 1.27 1.27)) (justify left bottom))
   )
-  (label "EX5" (at 24.765 48.26 0) (fields_autoplaced)
-    (effects (font (size 1.27 1.27)) (justify left bottom))
-  )
-  (label "MOSI" (at 184.15 144.145 0) (fields_autoplaced)
+  (label "SCK2" (at 24.765 45.72 0) (fields_autoplaced)
+    (effects (font (size 1.27 1.27)) (justify left bottom))
+  )
+  (label "MOSI2" (at 184.15 144.145 0) (fields_autoplaced)
     (effects (font (size 1.27 1.27)) (justify left bottom))
   )
@@
     (effects (font (size 1.27 1.27)) (justify left bottom))
   )
+  (label "SCK2" (at 73.025 88.265 0) (fields_autoplaced)
+    (effects (font (size 1.27 1.27)) (justify left bottom))
+  )
   (label "X1" (at 144.145 73.025 0) (fields_autoplaced)
     (effects (font (size 1.27 1.27)) (justify left bottom))
@@
     (effects (font (size 1.27 1.27)) (justify left bottom))
   )
-  (label "MISO" (at 184.15 146.685 0) (fields_autoplaced)
+  (label "MISO2" (at 184.15 146.685 0) (fields_autoplaced)
     (effects (font (size 1.27 1.27)) (justify left bottom))
   )
@@
     (effects (font (size 1.27 1.27)) (justify left bottom))
   )
-  (label "EX1" (at 24.765 43.18 0) (fields_autoplaced)
-    (effects (font (size 1.27 1.27)) (justify left bottom))
-  )
-  (label "SCK" (at 26.035 113.665 0) (fields_autoplaced)
+  (label "MOSI2" (at 24.765 43.18 0) (fields_autoplaced)
+    (effects (font (size 1.27 1.27)) (justify left bottom))
+  )
+  (label "SCK2" (at 26.035 113.665 0) (fields_autoplaced)
     (effects (font (size 1.27 1.27)) (justify left bottom))
   )
@@
     (effects (font (size 1.27 1.27)) (justify left bottom))
   )
-  (label "MOSI" (at 50.165 113.665 0) (fields_autoplaced)
-    (effects (font (size 1.27 1.27)) (justify left bottom))
-  )
+  (label "MOSI2" (at 50.165 113.665 0) (fields_autoplaced)
+    (effects (font (size 1.27 1.27)) (justify left bottom))
+  )
+  (label "MOSI2" (at 73.025 85.725 0) (fields_autoplaced)
+    (effects (font (size 1.27 1.27)) (justify left bottom))
+  )
